File: Cmoy Amp.sch (KiCad schematic (older format))
At the start: 12 parts, among them U1 OPA2132PA-ND

Commit message: Update PCB layout
Parts:
- renumbered JACK1 to JACK_IN1, JACK2 to JACK_OUT1
Changed lines of the file:
@@
 $EndComp
 $Comp
-L opa2132pa-nd:SJ1-3513 JACK1
+L opa2132pa-nd:SJ1-3513 JACK_IN1
 U 1 1 5A113486
 P 1275 6725
-F 0 "JACK1" H 1275 6125 98  0000 C CNN
+F 0 "JACK_IN1" H 1275 6125 98  0000 C CNN
 F 1 "SJ1-3513" H 1275 6325 118 0000 C CNN
 F 2 "MyLib:SJ1-3513" H 1275 6725 60  0001 C CNN
@@
 $EndComp
 $Comp
-L opa2132pa-nd:SJ1-3513 JACK2
+L opa2132pa-nd:SJ1-3513 JACK_OUT1
 U 1 1 5A113487
 P 3525 6675
-F 0 "JACK2" H 3525 6075 98  0000 C CNN
+F 0 "JACK_OUT1" H 3525 6075 98  0000 C CNN
 F 1 "SJ1-3513" H 3525 6275 118 0000 C CNN
 F 2 "MyLib:SJ1-3513" H 3525 6675 60  0001 C CNN
